Commit message: commit

File: openrov_description/urdf/sensors.xacro (robot description, xacro)
@@ -4,5 +4,5 @@
     Some examples of sensors that can be added to the vehicle frame.
     Set the origin of the sensor frames correctly for your application
-    Look into the sensor macros in the package uuv_sensor_ros_plugins/urdf for
+    Look igoogle traduornto the sensor macros in the package uuv_sensor_ros_plugins/urdf for
     more examples or add you own custom sensor units.
   -->
@@ -11,20 +11,4 @@
   <!-- Mount a Pose 3D sensor. -->
   <xacro:default_pose_3d namespace="${namespace}" parent_link="${namespace}/base_link" />
-  <!-- Forward-looking sonar sensor -->
-  <xacro:forward_multibeam_p900 namespace="${namespace}" parent_link="${namespace}/base_link">
-    <origin xyz="0 0 0" rpy="0 0 0"/>
-  </xacro:forward_multibeam_p900>
-  <!-- DVL  -->
-  <xacro:default_dvl namespace="${namespace}" parent_link="${namespace}/base_link">
-    <origin xyz="0 0 0" rpy="0 0 0"/>
-  </xacro:default_dvl>
-  <!-- RPT  -->
-  <xacro:default_rpt namespace="${namespace}" parent_link="${namespace}/base_link">
-    <origin xyz="0 0 0" rpy="0 0 0"/>
-  </xacro:default_rpt>
-  <!-- Pressure  -->
-  <xacro:default_pressure namespace="${namespace}" parent_link="${namespace}/base_link">
-    <origin xyz="0 0 0" rpy="0 0 0"/>
-  </xacro:default_pressure>
   <!-- IMU  -->
   <xacro:default_imu namespace="${namespace}" parent_link="${namespace}/base_link">
