Commit message: starting thruster manager

File: openrov_description/urdf/gazebo.xacro (robot description, xacro)
@@ -4,5 +4,5 @@
     <xacro:property name="openrov_cob" value="0 0 0"/>
     <!-- Vehicle's actual volume (Gazebo cannot compute the volume out of the mesh) -->
-    <xacro:property name="openrov_volume" value="5e-3"/>
+    <xacro:property name="openrov_volume" value="0.00107346790644"/>
     <!-- Describing the dimensions of the vehicle's bounding box -->
     <xacro:property name="openrov_length" value="0.30"/>
@@ -88,9 +88,9 @@
         </hydrodynamic_model>
         <!-- 2) This computes the added-mass and damping parameters for a sphere
-        in the fluid with the given radius -->
+        in the fluid with the given radius >
         <hydrodynamic_model>
           <type>sphere</type>
           <radius>0</radius>
-        </hydrodynamic_model>
+        </hydrodynamic_model-->
       </link>
     </xacro:macro>

File: openrov_description/urdf/snippets.xacro (robot description, xacro)
@@ -53,10 +53,10 @@
         <gain>1</gain>
         <!-- Maximum allowed input value for the input signal for thruster unit -->
-        <clampMax>0</clampMax>
+        <clampMax>100</clampMax>
         <!-- Minimum allowed value for the input signal for thruster unit -->
         <clampMin>0</clampMin>
         <!-- Minimum and maximum thrust force output allowed -->
         <thrustMin>0</thrustMin>
-        <thrustMax>0</thrustMax>
+        <thrustMax>100</thrustMax>
         <!--
         Value from 0 to 1 to set the efficiency of the output thrust force
@@ -81,8 +81,8 @@
         </dynamics>
         <!-- 2) First order model -->
-        <dynamics>
+        <!--dynamics>
           <type>FirstOrder</type>
           <timeConstant>0.0</timeConstant>
-        </dynamics>
+        </dynamics-->
         <!-- 3) Yoerger's nonlinear dynamic model
         For information on the model description:
@@ -92,9 +92,9 @@
             no. 3, pp. 167-178, Jul. 1990.
         -->
-        <dynamics>
+        <!--dynamics>
           <type>Yoerger</type>
           <alpha>0.0</alpha>
           <beta>0.0</beta>
-        </dynamics>
+        </dynamics-->
         <!-- 4) Bessa's nonlinear dynamic model
         For information on the model description:
@@ -104,5 +104,5 @@
             Mechatronics. Vol. 2. 2006.
         -->
-        <dynamics>
+        <!--dynamics>
           <type>Bessa</type>
           <Jmsp>0.0</Jmsp>
@@ -111,5 +111,5 @@
           <Kt>0.0</Kt>
           <Rm>0.0</Rm>
-        </dynamics>
+        </dynamics-->
         <!--
         Choose one of the model for the steady-state curve describing the
@@ -123,5 +123,5 @@
         <conversion>
           <type>Basic</type>
-          <rotorConstant>0.0</rotorConstant>
+          <rotorConstant>1.0</rotorConstant>
         </conversion>
         <!-- 2) Dead-zone nonlinearity described in Bessa, 2006
@@ -133,5 +133,5 @@
         thrust = rotorConstantR * (x * abs(x) - deltaR), if x * abs(x) >= deltaL
         -->
-        <conversion>
+        <!--conversion>
           <type>Bessa</type>
           <rotorConstantL>0.0</rotorConstantL>
@@ -139,5 +139,5 @@
           <deltaL>0.0</deltaL>
           <deltaR>0.0</deltaR>
-        </conversion>
+        </conversion-->
         <!-- 3) Linear interpolation
         If you have access to the thruster's data sheet, for example,
@@ -146,9 +146,9 @@
         of the given samples.
         -->
-        <conversion>
+        <!--conversion>
           <type>LinearInterp</type>
           <inputValues>0 1 2 3</inputValues>
           <outputValues>0 1 2 3</outputValues>
-        </conversion>
+        </conversion-->
       </plugin>
     </gazebo>
