Commit message: scaled urdf

File: openrov_description/urdf/actuators.xacro (robot description, xacro)
@@ -9,24 +9,15 @@
     -->
     <xacro:thruster_macro robot_namespace="${namespace}" thruster_id="0">
-        <origin xyz="0 0 0" rpy="0 0 ${pi}" />
+        <origin xyz="-0.069639 0.000293 0.058843 " rpy="0 ${pi/2} 0" />
     </xacro:thruster_macro>
     <xacro:thruster_macro robot_namespace="${namespace}" thruster_id="1">
-        <origin xyz="0 0 0" rpy="0 0 ${pi}" />
+        <origin xyz="-0.146087 0.04559  0" rpy="0 0 0" />
     </xacro:thruster_macro>
     <xacro:thruster_macro robot_namespace="${namespace}" thruster_id="2">
-    <origin xyz="0 0 0" rpy="0 -${0.5*pi} 0" />
+    <origin xyz="-0.146087 -0.044872 0" rpy="0 0 0" />
     </xacro:thruster_macro>
     <!-- Instantiate fins, if necessary -->
     <xacro:fin_macro namespace="${namespace}" fin_id="0">
-      <origin xyz="0 0 0" rpy="0 0 0" />
-    </xacro:fin_macro>
-    <xacro:fin_macro namespace="${namespace}" fin_id="1">
-      <origin xyz="0 0 0" rpy="0 0 0" />
-    </xacro:fin_macro>
-    <xacro:fin_macro namespace="${namespace}" fin_id="2">
-      <origin xyz="0 0 0" rpy="0 0 0" />
-    </xacro:fin_macro>
-    <xacro:fin_macro namespace="${namespace}" fin_id="3">
-      <origin xyz="0 0 0" rpy="0 0 0" />
+      <origin xyz="0.04687 -0.26058 0.20071" rpy="0 0 0" />
     </xacro:fin_macro>
 </robot>

File: openrov_description/urdf/base.xacro (robot description, xacro)
@@ -39,12 +39,12 @@
           <mass value="${mass}" />
           <origin xyz="${cog}" rpy="0 0 0"/>
-          <inertia ixx="0" ixy="0" ixz="0"
-                   iyy="0" iyz="0"
-                   izz="0" />
+          <inertia ixx="1" ixy="0" ixz="0"
+                   iyy="1" iyz="0"
+                   izz="1" />
         </inertial>
         <visual>
           <origin xyz="0 0 0" rpy="0 0 0"/>
           <geometry>
-            <mesh filename="${visual_mesh_file}" scale="1 1 1" />
+            <mesh filename="${visual_mesh_file}" scale="${scale}" />
           </geometry>
         </visual>
@@ -52,5 +52,5 @@
           <origin xyz="0 0 0" rpy="0 0 0"/>
           <geometry>
-            <mesh filename="${collision_mesh_file}" scale="1 1 1" />
+            <mesh filename="${collision_mesh_file}" scale="${scale}" />
           </geometry>
         </collision>

File: openrov_description/urdf/gazebo.xacro (robot description, xacro)
@@ -4,9 +4,9 @@
     <xacro:property name="openrov_cob" value="0 0 0"/>
     <!-- Vehicle's actual volume (Gazebo cannot compute the volume out of the mesh) -->
-    <xacro:property name="openrov_volume" value="0"/>
+    <xacro:property name="openrov_volume" value="5e-3"/>
     <!-- Describing the dimensions of the vehicle's bounding box -->
-    <xacro:property name="openrov_length" value="0"/>
-    <xacro:property name="openrov_width"  value="0"/>
-    <xacro:property name="openrov_height" value="0"/>
+    <xacro:property name="openrov_length" value="0.30"/>
+    <xacro:property name="openrov_width"  value="0.20"/>
+    <xacro:property name="openrov_height" value="0.15"/>
     <xacro:macro name="openrov_hydro_model" params="namespace">
       <!-- List of hydrodynamic models this robot's links -->

File: openrov_description/urdf/snippets.xacro (robot description, xacro)
@@ -1,4 +1,5 @@
 <?xml version="1.0"?>
 <robot xmlns:xacro="http://www.ros.org/wiki/xacro">
+  <xacro:property name="scale" value="1 1 1"/>
   <!--                                                                      -->
   <!-- MACRO FOR THRUSTER UNITS  -->
@@ -21,5 +22,5 @@
       <visual>
         <geometry>
-          <mesh filename="${prop_mesh_file}" scale="1 1 1" />
+          <mesh filename="${prop_mesh_file}" scale="${scale}" />
         </geometry>
       </visual>
@@ -187,5 +188,5 @@
           <origin xyz="0 0 0" rpy="0 0 0" />
           <geometry>
-            <mesh filename="${fin_mesh_file}" scale="1 1 1"/>
+            <mesh filename="${fin_mesh_file}" scale="${scale}"/>
           </geometry>
         </visual>
@@ -212,5 +213,5 @@
           <liftdrag>
             <type>TwoLines</type>
-            <area>${replace here the value for the area of the fin's cross section}</area>
+            <area>${0.000630}</area>
             <fluid_density>0.0</fluid_density>
             <a0>0.0</a0>

Commit message: no fin

File: openrov_description/urdf/actuators.xacro (robot description, xacro)
@@ -17,7 +17,3 @@
     <origin xyz="-0.146087 -0.044872 0" rpy="0 0 0" />
     </xacro:thruster_macro>
-    <!-- Instantiate fins, if necessary -->
-    <xacro:fin_macro namespace="${namespace}" fin_id="0">
-      <origin xyz="0.04687 -0.26058 0.20071" rpy="0 0 0" />
-    </xacro:fin_macro>
 </robot>

File: openrov_description/urdf/base.xacro (robot description, xacro)
@@ -14,5 +14,5 @@
   <xacro:property name="mass" value="2.6"/>
   <!-- Center of gravity -->
-  <xacro:property name="cog" value="0 0 0"/>
+  <xacro:property name="cog" value="0.005 0 0.01"/>
   <!-- Fluid density -->
   <xacro:property name="rho" value="1028"/>

File: openrov_description/urdf/snippets.xacro (robot description, xacro)
@@ -156,95 +156,3 @@
     </gazebo>
   </xacro:macro>
-  <!--                                                                      -->
-  <!-- MACRO FOR FIN/RUDDER UNITS  -->
-  <!--                                                                      -->
-  <!--
-    This macro can be used to add fins to the body of the vehicle, the fins
-    should be initialized in the actuators.xacro file. If you vehicle has no
-    fins, you can erase the macro below.
-  -->
-  <!-- A separate mesh for the fin should be stored in the meshes folder -->
-  <xacro:property name="fin_mesh_file" value="file://$(find openrov_description)/meshes/fin.dae"/>
-  <!-- Fin joint limits  -->
-  <xacro:property name="fin_min_joint_limit" value="${0.0 * d2r}"/>
-  <xacro:property name="fin_max_joint_limit" value="${0.0 * d2r}"/>
-  <xacro:macro name="fin_macro" params="namespace fin_id *origin">
-      <joint name="${namespace}/fin${fin_id}_joint" type="revolute">
-          <limit effort="0" lower="${fin_min_joint_limit}" upper="${fin_max_joint_limit}" velocity="0"/>
-          <xacro:insert_block name="origin"/>
-          <axis xyz="0 0 1"/>
-          <parent link="${namespace}/base_link" />
-          <child link="${namespace}/fin${fin_id}" />
-      </joint>
-      <link name="${namespace}/fin${fin_id}">
-        <inertial>
-          <mass value="0.001" />
-          <origin xyz="0 0 0" rpy="0 0 0"/>
-          <inertia ixx="0.000000017" ixy="0.0" ixz="0.0"
-                 iyy="0.000000017" iyz="0.0"
-                 izz="0.000000017" />
-        </inertial>
-        <visual>
-          <origin xyz="0 0 0" rpy="0 0 0" />
-          <geometry>
-            <mesh filename="${fin_mesh_file}" scale="${scale}"/>
-          </geometry>
-        </visual>
-      </link>
-      <gazebo>
-        <plugin name="${namespace}_fin${fin_id}_model" filename="libuuv_fin_ros_plugin.so">
-          <!--
-            First order dynamics model for the fin joint dynamics,
-            replace an appropriate time constant
-          -->
-          <dynamics>
-            <type>FirstOrder</type>
-            <timeConstant>0.0</timeConstant>
-          </dynamics>
-          <!--
-            Definition of the lift and drag model, choose ONE of the models
-            below according to the model you want to use.
-          -->
-          <!--
-            1) References for the two line lift and drag model:
-              [1] https://en.wikipedia.org/wiki/Lift_coefficient
-              [2] http://gazebosim.org/tutorials?tut=aerodynamics&cat=plugins
-          -->
-          <liftdrag>
-            <type>TwoLines</type>
-            <area>${0.000630}</area>
-            <fluid_density>0.0</fluid_density>
-            <a0>0.0</a0>
-            <alpha_stall>0.0</alpha_stall>
-            <cla>0.0</cla><!-- ^= 0.244 when using deg -->
-            <cla_stall>0.0</cla_stall>
-            <cda>0.0</cda>
-            <cda_stall>0.0</cda_stall>
-          </liftdrag>
-          <!--
-            2) Reference for the quadratic lift and drag model:
-              [1] Engelhardtsen, Oystein. 3D AUV Collision Avoidance.
-                  MS thesis. Institutt for teknisk kybernetikk, 2007.
-                  https://brage.bibsys.no/xmlui/handle/11250/259834
-          -->
-          <liftdrag>
-            <type>Quadratic</type>
-            <lift_constant>0.0</lift_constant>
-            <drag_constant>0.0</drag_constant>
-          </liftdrag>
-          <!--
-            Further parameters necessary for the lift and drag plugin
-          -->
-          <!-- Current velocity topic -->
-          <current_velocity_topic>/hydrodynamics/current_velocity</current_velocity_topic>
-          <!-- Name of the correspodent fin link and joint  -->
-          <link_name>${namespace}/fin${fin_id}</link_name>
-          <joint_name>${namespace}/fin${fin_id}_joint</joint_name>
-          <!-- Output topic to publish the current angle of the fin joint -->
-          <output_topic>${namespace}/fins/${fin_id}/output</output_topic>
-          <input_topic>${namespace}/fins/${fin_id}/input</input_topic>
-          <wrench_topic>${namespace}/fins/${fin_id}/wrench_topic</wrench_topic>
-        </plugin>
-      </gazebo>
-  </xacro:macro>
 </robot>

Commit message: finishing urdf

File: openrov_description/urdf/actuators.xacro (robot description, xacro)
@@ -9,11 +9,11 @@
     -->
     <xacro:thruster_macro robot_namespace="${namespace}" thruster_id="0">
-        <origin xyz="-0.069639 0.000293 0.058843 " rpy="0 ${pi/2} 0" />
+        <origin xyz="-0.062 0 0.062" rpy="0 ${-PI/2} 0"/>
     </xacro:thruster_macro>
     <xacro:thruster_macro robot_namespace="${namespace}" thruster_id="1">
-        <origin xyz="-0.146087 0.04559  0" rpy="0 0 0" />
+        <origin xyz="-0.14 -0.045 0" rpy="0 0 ${PI}"/>
     </xacro:thruster_macro>
     <xacro:thruster_macro robot_namespace="${namespace}" thruster_id="2">
-    <origin xyz="-0.146087 -0.044872 0" rpy="0 0 0" />
+    <origin xyz="-0.14 0.045 0" rpy="0 0 ${PI}"/>
     </xacro:thruster_macro>
 </robot>

File: openrov_description/urdf/base.xacro (robot description, xacro)
@@ -4,5 +4,6 @@
   <xacro:include filename="$(find uuv_descriptions)/urdf/common.urdf.xacro"/>
   <!-- Loading file with sensor macros -->
-  <xacro:include filename="$(find uuv_sensor_ros_plugins)/urdf/sensor_snippets.xacro"/>
+  <!--xacro:include filename="$(find uuv_sensor_ros_plugins)/urdf/sensor_snippets.xacro"/-->
+  <!--xacro:include filename="$(find openrov_description)/urdf/sensor_snippets.xacro"/-->
   <!-- Loading the UUV simulator ROS plugin macros -->
   <xacro:include filename="$(find uuv_gazebo_ros_plugins)/urdf/snippets.xacro"/>
@@ -12,7 +13,7 @@
     Vehicle's parameters (remember to enter the model parameters below)
   -->
-  <xacro:property name="mass" value="2.6"/>
+  <xacro:property name="mass" value="2.4"/>
   <!-- Center of gravity -->
-  <xacro:property name="cog" value="0.005 0 0.01"/>
+  <xacro:property name="cog" value="0.0 0.0 0.0"/>
   <!-- Fluid density -->
   <xacro:property name="rho" value="1028"/>
@@ -27,5 +28,5 @@
   this geometry as simple as possible to improve the performance the physics engine
   regarding the computation of collision forces) -->
-  <xacro:property name="collision_mesh_file" value="file://$(find openrov_description)/meshes/vehicle.stl"/>
+  <!--xacro:property name="collision_mesh_file" value="file://$(find openrov_description)/meshes/vehicle.stl"/-->
   <!-- Vehicle macro -->
   <xacro:macro name="openrov_base" params="namespace *gazebo">
@@ -39,7 +40,7 @@
           <mass value="${mass}" />
           <origin xyz="${cog}" rpy="0 0 0"/>
-          <inertia ixx="1" ixy="0" ixz="0"
-                   iyy="1" iyz="0"
-                   izz="1" />
+          <inertia ixx="0.01355" ixy="0" ixz="0"
+                   iyy="0.00480" iyz="0"
+                   izz="0.00593" />
         </inertial>
         <visual>
@@ -52,5 +53,6 @@
           <origin xyz="0 0 0" rpy="0 0 0"/>
           <geometry>
-            <mesh filename="${collision_mesh_file}" scale="${scale}" />
+            <!--mesh filename="${collision_mesh_file}" scale="${scale}" /-->
+            <box size="0.30 0.20 0.15"/>
           </geometry>
         </collision>
@@ -64,5 +66,5 @@
     <xacro:include filename="$(find openrov_description)/urdf/actuators.xacro"/>
     <!-- Include the sensor modules -->
-    <xacro:include filename="$(find openrov_description)/urdf/sensors.xacro"/>
+    <!--xacro:include filename="$(find openrov_description)/urdf/sensors.xacro"/\-->
   </xacro:macro>
 </robot>

File: openrov_description/urdf/sensors.xacro (robot description, xacro)
@@ -1,21 +1,6 @@
 <?xml version="1.0"?>
 <robot xmlns:xacro="http://www.ros.org/wiki/xacro">
-  <!--
-    Some examples of sensors that can be added to the vehicle frame.
-    Set the origin of the sensor frames correctly for your application
-    Look igoogle traduornto the sensor macros in the package uuv_sensor_ros_plugins/urdf for
-    more examples or add you own custom sensor units.
-  -->
-  <!-- Mount a GPS. -->
-  <xacro:default_gps namespace="${namespace}" parent_link="${namespace}/base_link" />
-  <!-- Mount a Pose 3D sensor. -->
-  <xacro:default_pose_3d namespace="${namespace}" parent_link="${namespace}/base_link" />
-  <!-- IMU  -->
-  <xacro:default_imu namespace="${namespace}" parent_link="${namespace}/base_link">
-    <origin xyz="0 0 0" rpy="0 0 0"/>
-  </xacro:default_imu>
-  <!-- Mount a camera  -->
-  <xacro:default_camera namespace="${namespace}" parent_link="${namespace}/base_link" suffix="">
-    <origin xyz="0 0 0" rpy="0 0 0"/>
+  <xacro:default_camera namespace="${namespace}" parent_link="${namespace}/base_link">
+    <origin xyz="0.05 0 0" rpy="0 0 0"/>
   </xacro:default_camera>
 </robot>

File: openrov_description/urdf/snippets.xacro (robot description, xacro)
@@ -2,4 +2,5 @@
 <robot xmlns:xacro="http://www.ros.org/wiki/xacro">
   <xacro:property name="scale" value="1 1 1"/>
+  <xacro:property name="PI" value="3.1415926"/>
   <!--                                                                      -->
   <!-- MACRO FOR THRUSTER UNITS  -->

Commit message: keyboard and joystick control implemented. Adjusting parameters

File: openrov_description/urdf/actuators.xacro (robot description, xacro)
@@ -8,11 +8,11 @@
           aware that Gazebo does not use the SNAME convention per default.
     -->
-    <xacro:thruster_macro robot_namespace="${namespace}" thruster_id="0">
+    <xacro:thruster_macro namespace="${namespace}" thruster_id="0">
         <origin xyz="-0.062 0 0.062" rpy="0 ${-PI/2} 0"/>
     </xacro:thruster_macro>
-    <xacro:thruster_macro robot_namespace="${namespace}" thruster_id="1">
+    <xacro:thruster_macro namespace="${namespace}" thruster_id="1">
         <origin xyz="-0.14 -0.045 0" rpy="0 0 ${PI}"/>
     </xacro:thruster_macro>
-    <xacro:thruster_macro robot_namespace="${namespace}" thruster_id="2">
+    <xacro:thruster_macro namespace="${namespace}" thruster_id="2">
     <origin xyz="-0.14 0.045 0" rpy="0 0 ${PI}"/>
     </xacro:thruster_macro>

File: openrov_description/urdf/snippets.xacro (robot description, xacro)
@@ -10,21 +10,9 @@
   -->
   <xacro:property name="prop_mesh_file" value="file://$(find openrov_description)/meshes/propeller.dae"/>
-  <!-- Thruster joint and link snippet -->
-  <xacro:macro name="thruster_macro"
-    params="namespace thruster_id *origin">
-    <xacro:thruster_module_first_order_basic_fcn_macro
-      namespace="${namespace}"
-      thruster_id="${thruster_id}"
-      mesh_filename="$(prop_mesh_file)"
-      dyn_time_constant="0.05"
-      rotor_constant="0.026546">
-      <xacro:insert_block name="origin"/>
-    </xacro:thruster_module_first_order_basic_fcn_macro>
-  </xacro:macro>
   <!--
     Thruster macro with integration of joint and link. The thrusters should
     be initialized in the actuators.xacro file.
   -->
-  <!--xacro:macro name="thruster_macro" params="robot_namespace thruster_id *origin">
+  <xacro:macro name="thruster_macro" params="namespace thruster_id *origin">
     <!--
     Dummy link as place holder for the thruster frame,
@@ -32,5 +20,5 @@
     of the vehicle and may cause internal collisions if set otherwise
     -->
-    <link name="${robot_namespace}/thruster_${thruster_id}">
+    <link name="${namespace}/thruster_${thruster_id}">
       <visual>
         <geometry>
@@ -47,27 +35,26 @@
     </link>
     <!-- Joint between thruster link and vehicle base link -->
-    <joint name="${robot_namespace}/thruster_${thruster_id}_joint" type="continuous">
+    <joint name="${namespace}/thruster_${thruster_id}_joint" type="continuous">
       <xacro:insert_block name="origin" />
       <axis xyz="1 0 0" />
-      <parent link="${robot_namespace}/base_link" />
-      <child link="${robot_namespace}/thruster_${thruster_id}" />
+      <parent link="${namespace}/base_link" />
+      <child link="${namespace}/thruster_${thruster_id}" />
     </joint>
     <gazebo>
       <!-- Thruster ROS plugin -->
-      <plugin name="${robot_namespace}_${thruster_id}_thruster_model" filename="libuuv_thruster_ros_plugin.so">
+      <plugin name="${namespace}_${thruster_id}_thruster_model" filename="libuuv_thruster_ros_plugin.so">
         <!-- Name of the thruster link -->
-        <linkName>${robot_namespace}/thruster_${thruster_id}</linkName>
+        <linkName>${namespace}/thruster_${thruster_id}</linkName>
         <!-- Name of the joint between thruster and vehicle base link -->
-        <jointName>${robot_namespace}/thruster_${thruster_id}_joint</jointName>
+        <jointName>${namespace}/thruster_${thruster_id}_joint</jointName>
         <!-- Make the thruster aware of its id -->
         <thrusterID>${thruster_id}</thrusterID>
         <!-- Gain of the input command signal -->
         <gain>1</gain>
-        <!-- Maximum allowed input value for the input signal for thruster unit -->
+        <!-- Minimum and maximum allowed input value for the input signal for thruster unit -->
+        <clampMin>-100</clampMin>
         <clampMax>100</clampMax>
-        <!-- Minimum allowed value for the input signal for thruster unit -->
-        <clampMin>0</clampMin>
         <!-- Minimum and maximum thrust force output allowed -->
-        <thrustMin>0</thrustMin>
+        <thrustMin>-100</thrustMin>
         <thrustMax>100</thrustMax>
         <!--
@@ -165,7 +152,7 @@
       </plugin>
     </gazebo>
-    <gazebo reference="${robot_namespace}/thruster_${thruster_id}">
+    <gazebo reference="${namespace}/thruster_${thruster_id}">
       <selfCollide>false</selfCollide>
     </gazebo>
-  </xacro:macro-->
+  </xacro:macro>
 </robot>

Commit message: pkg openrov_teleop created

File: openrov_description/urdf/actuators.xacro (robot description, xacro)
@@ -15,5 +15,5 @@
     </xacro:thruster_macro>
     <xacro:thruster_macro namespace="${namespace}" thruster_id="2">
-    <origin xyz="-0.14 0.045 0" rpy="0 0 ${PI}"/>
+        <origin xyz="-0.14 0.045 0" rpy="0 0 ${PI}"/>
     </xacro:thruster_macro>
 </robot>

File: openrov_description/urdf/gazebo.xacro (robot description, xacro)
@@ -2,5 +2,5 @@
 <robot xmlns:xacro="http://www.ros.org/wiki/xacro">
     <!-- Center of buoyancy -->
-    <xacro:property name="openrov_cob" value="0 0 0"/>
+    <xacro:property name="openrov_cob" value="0.004 0 0.009"/>
     <!-- Vehicle's actual volume (Gazebo cannot compute the volume out of the mesh) -->
     <xacro:property name="openrov_volume" value="0.00107346790644"/>
