Commit message: urdf done. Adding plugins

File: openrov_description/urdf/base.xacro (robot description, xacro)
@@ -4,6 +4,6 @@
   <xacro:include filename="$(find uuv_descriptions)/urdf/common.urdf.xacro"/>
   <!-- Loading file with sensor macros -->
-  <!--xacro:include filename="$(find uuv_sensor_ros_plugins)/urdf/sensor_snippets.xacro"/-->
-  <!--xacro:include filename="$(find openrov_description)/urdf/sensor_snippets.xacro"/-->
+  <xacro:include filename="$(find uuv_sensor_ros_plugins)/urdf/pose_3d_snippets.xacro"/>
+  <xacro:include filename="$(find openrov_description)/urdf/sensor_snippets.xacro"/>
   <!-- Loading the UUV simulator ROS plugin macros -->
   <xacro:include filename="$(find uuv_gazebo_ros_plugins)/urdf/snippets.xacro"/>
@@ -66,5 +66,5 @@
     <xacro:include filename="$(find openrov_description)/urdf/actuators.xacro"/>
     <!-- Include the sensor modules -->
-    <!--xacro:include filename="$(find openrov_description)/urdf/sensors.xacro"/\-->
+    <xacro:include filename="$(find openrov_description)/urdf/sensors.xacro"/>
   </xacro:macro>
 </robot>

File: openrov_description/urdf/sensor_snippets.xacro (robot description, xacro)
@@ -1,33 +1,98 @@
 <?xml version="1.0"?>
 <robot xmlns:xacro="http://www.ros.org/wiki/xacro">
-  <xacro:macro name="default_camera" params="namespace parent_link *origin">
+  <xacro:property name="meshes_path" value="$(find openrov_description)/meshes"/>
+  <xacro:macro name="camera_openrov" params="namespace parent_link *origin">
     <link name="${namespace}/camera_link">
       <visual>
         <origin xyz="0.0 0.0 0.0" rpy="0.0 0.0 0.0"/>
         <geometry>
-          <mesh filename="${meshes_path}/camera.dae" scale="${scale}"/>
+          <mesh filename="${meshes_path}/camera.dae"/>
         </geometry>
       </visual>
+      <inertial>
+        <origin xyz="0.0 0.0 0.0" rpy="0.0 0.0 0.0"/>
+        <mass value="0.001"/>
+        <inertia ixx="0.00000001" ixy="0.0" ixz="0.0" iyy="0.00000001" iyz="0.0" izz="0.00000001"/>
+      </inertial>
     </link>
     <link name="${namespace}/camera_fix">
       <visual>
-        <xacro:insert_block name="origin">
+        <xacro:insert_block name="origin"/>
         <geometry>
           <box size="0.01 0.01 0.01"/>
         </geometry>
       </visual>
+      <inertial>
+        <origin xyz="0.0 0.0 0.0" rpy="0.0 0.0 0.0"/>
+        <mass value="0.001"/>
+        <inertia ixx="0.00000001" ixy="0.0" ixz="0.0" iyy="0.00000001" iyz="0.0" izz="0.00000001"/>
+      </inertial>
     </link>
     <joint name="${namespace}/camera_to_fix" type="fixed">
-      <xacro:insert_block name="origin">
-      <parent link="camera_fix"/>
-      <child link="camera_link"/>
+      <xacro:insert_block name="origin"/>
+      <parent link="${namespace}/camera_fix"/>
+      <child link="${namespace}/camera_link"/>
     </joint>
     <joint name="${namespace}/base_to_camera" type="revolute">
       <origin xyz="0.025 0.0 0.015419" rpy="0.0 0.0 0.0"/>
-      <parent link="base_link"/>
-      <child link="camera_fix"/>
+      <parent link="${parent_link}"/>
+      <child link="${namespace}/camera_fix"/>
       <axis xyz="0 1 0"/>
       <limit lower="${-PI/4}" upper="${PI/4}" effort="0.0" velocity="0.0"/>
     </joint>
+    <gazebo reference="${namespace}/camera_link">
+      <sensor type="camera" name="camera">
+        <update_rate>30.0</update_rate>
+        <camera name="head">
+          <horizontal_fov>2.0944</horizontal_fov>
+          <image>
+            <width>1280</width>
+            <height>720</height>
+            <format>R8G8B8</format>
+          </image>
+          <clip>
+            <near>0.02</near>
+            <far>300</far>
+          </clip>
+          <noise>
+            <type>gaussian</type>
+            <!-- Noise is sampled independently per pixel on each frame.
+                 That pixel's noise value is added to each of its color
+                 channels, which at that point lie in the range [0,1]. -->
+            <mean>0.0</mean>
+            <stddev>0.007</stddev>
+          </noise>
+        </camera>
+        <plugin name="camera_controller" filename="libgazebo_ros_camera.so">
+          <alwaysOn>true</alwaysOn>
+          <updateRate>0.0</updateRate>
+          <cameraName>${namespace}/camera</cameraName>
+          <imageTopicName>image_raw</imageTopicName>
+          <cameraInfoTopicName>camera_info</cameraInfoTopicName>
+          <frameName>camera_link</frameName>
+          <hackBaseline>0.07</hackBaseline>
+          <distortionK1>0.0</distortionK1>
+          <distortionK2>0.0</distortionK2>
+          <distortionK3>0.0</distortionK3>
+          <distortionT1>0.0</distortionT1>
+          <distortionT2>0.0</distortionT2>
+        </plugin>
+      </sensor>
+    </gazebo>
+    <transmission name="tran_cam">
+      <type>transmission_interface/SimpleTransmission</type>
+      <joint name="${namespace}/base_to_camera">
+        <hardwareInterface>EffortJointInterface</hardwareInterface>
+      </joint>
+      <actuator name="motor_cam">
+        <hardwareInterface>EffortJointInterface</hardwareInterface>
+        <mechanicalReduction>1</mechanicalReduction>
+      </actuator>
+    </transmission>
+    <gazebo>
+      <plugin name="gazebo_ros_control" filename="libgazebo_ros_control.so">
+        <robotNamespace>/${namespace}</robotNamespace>
+      </plugin>
+    </gazebo>
   </xacro:macro>
 </robot>

File: openrov_description/urdf/sensors.xacro (robot description, xacro)
@@ -1,6 +1,9 @@
 <?xml version="1.0"?>
 <robot xmlns:xacro="http://www.ros.org/wiki/xacro">
-  <xacro:default_camera namespace="${namespace}" parent_link="${namespace}/base_link">
+  <!-- Mount a camera. -->
+  <xacro:camera_openrov namespace="${namespace}" parent_link="${namespace}/base_link">
     <origin xyz="0.05 0 0" rpy="0 0 0"/>
-  </xacro:default_camera>
+  </xacro:camera_openrov>
+  <!-- Mount a Pose 3D sensor. -->
+  <xacro:default_pose_3d namespace="${namespace}" parent_link="${namespace}/base_link" />
 </robot>

Commit message: volume and inertia matrix updated

File: openrov_description/urdf/base.xacro (robot description, xacro)
@@ -13,5 +13,5 @@
     Vehicle's parameters (remember to enter the model parameters below)
   -->
-  <xacro:property name="mass" value="2.4"/>
+  <xacro:property name="mass" value="2.47"/>
   <!-- Center of gravity -->
   <xacro:property name="cog" value="0.0 0.0 0.0"/>
@@ -40,7 +40,7 @@
           <mass value="${mass}" />
           <origin xyz="${cog}" rpy="0 0 0"/>
-          <inertia ixx="0.01355" ixy="0" ixz="0"
-                   iyy="0.00480" iyz="0"
-                   izz="0.00593" />
+          <inertia ixx="1.752e-2" ixy="1.593e-5" ixz="1.803e-3"
+                   iyy="1.265e-2" iyz="2.172e-5"
+                   izz="2.141e-2" />
         </inertial>
         <visual>

File: openrov_description/urdf/gazebo.xacro (robot description, xacro)
@@ -4,5 +4,5 @@
     <xacro:property name="openrov_cob" value="0.004 0 0.009"/>
     <!-- Vehicle's actual volume (Gazebo cannot compute the volume out of the mesh) -->
-    <xacro:property name="openrov_volume" value="0.00107346790644"/>
+    <xacro:property name="openrov_volume" value="0.0024"/>
     <!-- Describing the dimensions of the vehicle's bounding box -->
     <xacro:property name="openrov_length" value="0.30"/>

Commit message: writing openrov_control.rviz

File: openrov_description/urdf/base.xacro (robot description, xacro)
@@ -15,5 +15,6 @@
   <xacro:property name="mass" value="2.47"/>
   <!-- Center of gravity -->
-  <xacro:property name="cog" value="0.0 0.0 0.0"/>
+  <!--xacro:property name="cog" value="0.0 0.0 0.0"/-->
+  <xacro:property name="cog" value="-0.062 0 0.062"/>
   <!-- Fluid density -->
   <xacro:property name="rho" value="1028"/>
