Commit message: thruster snippets changed

File: openrov_description/robots/default.xacro (robot description, xacro)
@@ -28,4 +28,4 @@
   </xacro:openrov_base>
   <!-- Joint state publisher plugin -->
-  <xacro:default_joint_state_publisher namespace="$(arg namespace)" update_rate="10"/>
+  <xacro:default_joint_state_publisher namespace="$(arg namespace)" update_rate="50"/>
 </robot>

File: openrov_description/urdf/gazebo.xacro (robot description, xacro)
@@ -57,7 +57,7 @@
             This matrix is mostly useful for slender bodies (e.g. AUVs with torpedo shape)
           -->
-          <linear_damping_forward_speed>
+          <!--linear_damping_forward_speed>
             0 0 0 0 0 0
-          </linear_damping_forward_speed>
+          </linear_damping_forward_speed-->
           <!--
             The quadratic damping coefficients can be provided as a diagonal (6 elements)

File: openrov_description/urdf/sensor_snippets.xacro (robot description, xacro)
@@ -80,5 +80,5 @@
       </sensor>
     </gazebo>
-    <transmission name="tran_cam">
+    <!--transmission name="tran_cam">
       <type>transmission_interface/SimpleTransmission</type>
       <joint name="${namespace}/base_to_camera">
@@ -89,5 +89,5 @@
         <mechanicalReduction>1</mechanicalReduction>
       </actuator>
-    </transmission>
+    </transmission-->
     <gazebo>
       <plugin name="gazebo_ros_control" filename="libgazebo_ros_control.so">

File: openrov_description/urdf/snippets.xacro (robot description, xacro)
@@ -10,9 +10,21 @@
   -->
   <xacro:property name="prop_mesh_file" value="file://$(find openrov_description)/meshes/propeller.dae"/>
+  <!-- Thruster joint and link snippet -->
+  <xacro:macro name="thruster_macro"
+    params="namespace thruster_id *origin">
+    <xacro:thruster_module_first_order_basic_fcn_macro
+      namespace="${namespace}"
+      thruster_id="${thruster_id}"
+      mesh_filename="$(prop_mesh_file)"
+      dyn_time_constant="0.05"
+      rotor_constant="0.026546">
+      <xacro:insert_block name="origin"/>
+    </xacro:thruster_module_first_order_basic_fcn_macro>
+  </xacro:macro>
   <!--
     Thruster macro with integration of joint and link. The thrusters should
     be initialized in the actuators.xacro file.
   -->
-  <xacro:macro name="thruster_macro" params="robot_namespace thruster_id *origin">
+  <!--xacro:macro name="thruster_macro" params="robot_namespace thruster_id *origin">
     <!--
     Dummy link as place holder for the thruster frame,
@@ -156,4 +168,4 @@
       <selfCollide>false</selfCollide>
     </gazebo>
-  </xacro:macro>
+  </xacro:macro-->
 </robot>
